Commit message: Added flattened turtle (2 layers)

File: turtlebot3_description/urdf/turtlebot3_waffle_pi.gazebo.xacro (robot description, xacro)
@@ -2,6 +2,6 @@
 <robot name="turtlebot3_waffle_pi_sim" xmlns:xacro="http://ros.org/wiki/xacro">
   <xacro:arg name="laser_visual"  default="false"/>
-  <xacro:arg name="camera_visual" default="false"/>
-  <xacro:arg name="imu_visual"    default="false"/>
+  <xacro:arg name="camera_visual" default="true"/>
+  <xacro:arg name="imu_visual"    default="true"/>
   <gazebo reference="base_link">
     <material>Gazebo/DarkGrey</material>
@@ -142,6 +142,6 @@
           <horizontal_fov>1.085595</horizontal_fov>
           <image>
-              <width>640</width>
-              <height>480</height>
+              <width>720</width>
+              <height>640</height>
               <format>R8G8B8</format>
           </image>
@@ -156,5 +156,5 @@
         <cameraName>camera</cameraName>
         <frameName>camera_rgb_optical_frame</frameName>
-        <imageTopicName>rgb/image_raw</imageTopicName>
+        <imageTopicName>rgb/image</imageTopicName>
         <cameraInfoTopicName>rgb/camera_info</cameraInfoTopicName>
         <hackBaseline>0.07</hackBaseline>

File: turtlebot3_description/urdf/turtlebot3_waffle_pi.urdf.xacro (robot description, xacro)
@@ -13,12 +13,12 @@
       <origin xyz="-0.064 0 0.0" rpy="0 0 0"/>
       <geometry>
-        <mesh filename="package://turtlebot3_description/meshes/bases/waffle_pi_base.stl" scale="0.001 0.001 0.001"/>
+        <mesh filename="package://turtlebot3_description/meshes/bases/waffle_pi_base_flatten.stl" scale="0.001 0.001 0.001"/>
       </geometry>
       <material name="light_black"/>
     </visual>
     <collision>
-      <origin xyz="-0.064 0 0.047" rpy="0 0 0"/>
+      <origin xyz="-0.064 0 0.0295" rpy="0 0 0"/>
       <geometry>
-        <box size="0.266 0.266 0.094"/>
+        <box size="0.266 0.266 0.059"/>
       </geometry>
     </collision>
@@ -136,5 +136,5 @@
     <parent link="base_link"/>
     <child link="base_scan"/>
-    <origin xyz="-0.064 0 0.122" rpy="0 0 0"/>
+    <origin xyz="-0.064 0 0.087" rpy="0 0 3.14"/>
   </joint>
   <link name="base_scan">
@@ -161,5 +161,5 @@
   </link>
   <joint name="camera_joint" type="fixed">
-    <origin xyz="0.073 -0.011 0.084" rpy="0 0 0"/>
+    <origin xyz="0.073 -0.011 0.024" rpy="0 0 0"/>
     <parent link="base_link"/>
     <child link="camera_link"/>
@@ -167,5 +167,5 @@
   <link name="camera_link">
     <collision>
-      <origin xyz="0.005 0.011 0.013" rpy="0 0 0"/>
+      <origin xyz="0.005 0.011 0.013" rpy="1.57 0 0"/>
       <geometry>
         <box size="0.015 0.030 0.027"/>
